File: pcb-svetla-mn98.kicad_pcb (KiCad board)
At the start: 2 copper layers, 30 x 40 mm, 17 parts, among them J1 L TURN FRONT, J10 HEADLIGHT R, J11 MARKER R, J12 REAR RED R, J13 SPARE DRL, J14 P6DC INPUT, J2 R TURN FRONT, J3 L TURN REAR, J4 R TURN REAR, J5 SPARE FLASH, J6 HEADLIGHT L, J7 MARKER L, J8 REAR RED L, J9 ROOF RAMP

Commit message: Align J14 pinout with P6DC outputs
Connections:
- J14 pad 6: BACK-UP -> FLASH
- J14 pad 7: DRL -> BACK-UP
- J14 pad 8: FLASH -> DRL
Routing:
- net FLASH: track 90.5 -> 86.6 mm
- net DRL: track 114.1 -> 116.0 mm
- net BACK-UP: track 34.2 -> 36.2 mm
Other:
- board text added: "P6DC: 1/2 +, 3 L, 4 R, 5 B, 6 FLASH, 7 REV, 8 DRL"
- board text removed: "P6DC: 1/2 +, 3 L, 4 R, 5 B, 6 REV, 7 DRL, 8 FLASH"

Commit message: Keep J14 within board outline
Parts:
- moved J14 19.1 mm to (27.0, 36.3)
Routing:
- net DRL: track 116.0 -> 97.1 mm
- net FLASH: track 86.6 -> 67.8 mm
- net BACK-UP: track 36.2 -> 17.7 mm
- net BRAKE: track 32.4 -> 18.4 mm
- net LEFT: track 49.8 -> 59.8 mm
- net COMMON+: track 196.3 -> 200.1 mm
- net RIGHT: track 53.4 -> 56.9 mm

Commit message: Add synchronized KiCad schematic
Parts:
- J1, J10, J11, J12, J13, J2, J3, J4, J5, J6, J7, J8, J9: footprint JST_PH_S2B-PH-K_1x02_P2.00mm_Horizontal -> Connector_JST:JST_PH_S2B-PH-K_1x02_P2.00mm_Horizontal
- J14: footprint JST_PH_S8B-PH-K_1x08_P2.00mm_Horizontal -> Connector_JST:JST_PH_S8B-PH-K_1x08_P2.00mm_Horizontal
- JP1, JP3: footprint PinHeader_1x03_P2.54mm_Horizontal -> Connector_PinHeader_2.54mm:PinHeader_1x03_P2.54mm_Horizontal
- JP2: footprint PinHeader_2x03_P2.54mm_Vertical -> Connector_PinHeader_2.54mm:PinHeader_2x03_P2.54mm_Vertical
Connections:
- net BACK-UP renamed /BACK-UP
- net BRAKE renamed /BRAKE
- net COMMON+ renamed /COMMON+
- net DRL renamed /DRL
- net FLASH renamed /FLASH
- net LEFT renamed /LEFT
- net MARKER renamed /MARKER
- net RAMP renamed /RAMP
- net REAR_RED renamed /REAR_RED
- net RIGHT renamed /RIGHT
Routing:
- net (no net): track 0.00 -> 717.2 mm
- net /COMMON+: track 200.1 -> 0.00 mm
- net /DRL: track 97.1 -> 0.00 mm
- net /REAR_RED: track 76.2 -> 0.00 mm
- net /MARKER: track 71.0 -> 0.00 mm
- net /FLASH: track 67.8 -> 0.00 mm
- net /LEFT: track 59.8 -> 0.00 mm
- net /RIGHT: track 56.9 -> 0.00 mm
- net /RAMP: track 52.1 -> 0.00 mm
- net /BRAKE: track 18.4 -> 0.00 mm
- net /BACK-UP: track 17.7 -> 0.00 mm
